File: Power.sch (KiCad schematic (older format))
At the start: 17 parts

Commit message: File structure cleanup.
Parts:
- removed U?: AD2S1210, Package_QFP:LQFP-48-1EP_7x7mm_P0.5mm_EP3.6x3.6mm, symbol Resolver:AD2S1210
- added U?: AD2S1210, Package_QFP:LQFP-48-1EP_7x7mm_P0.5mm_EP3.6x3.6mm, symbol Resolver:AD2S1210
Connections:
- net +2V5: now also U?.47 (REFOUT)
- net +3V3: now also U?.18 (Vdrive)
- net +5V: now also U?.43 (AVdd), U?.6 (DVdd)
- net GND: now also U?.19 (DGND), U?.40 (AGND), U?.5 (DGND)
- net at C?.1, C?.1: now also U?.46 (REFBYP)
Changed lines of the file:
@@
 EESchema Schematic File Version 4
-LIBS:Main-cache
+LIBS:power
+LIBS:device
+LIBS:74xx
+LIBS:audio
+LIBS:interface
+LIBS:resolver-cache
 EELAYER 30 0
 EELAYER END
@@
 F 3 "" H 6450 2950 50  0001 C CNN
 	1    6450 2950
-	1    0    0    -1
-$EndComp
-$Comp
-L Resolver:AD2S1210 U?
-U 2 1 5EF0E7FF
-P 7400 2450
-F 0 "U?" H 7700 2950 50  0000 L CNN
-F 1 "AD2S1210" H 7550 2850 50  0000 L CNN
-F 2 "Package_QFP:LQFP-48-1EP_7x7mm_P0.5mm_EP3.6x3.6mm" H 9900 2200 50  0001 C CNN
-F 3 "https://www.analog.com/media/en/technical-documentation/data-sheets/AD2S1210.pdf" H 9900 2200 50  0001 C CNN
-	2    7400 2450
 	1    0    0    -1
 $EndComp
@@
 Text Notes 6400 1400 0    50   ~ 10
 Ei boi ska vi byta till 5VA och 5VD som referensdesignen?
+$Comp
+L Resolver:AD2S1210 U?
+U 2 1 5EE2BE29
+P 7400 2450
+F 0 "U?" H 7700 2950 50  0000 L CNN
+F 1 "AD2S1210" H 7600 2850 50  0000 L CNN
+F 2 "Package_QFP:LQFP-48-1EP_7x7mm_P0.5mm_EP3.6x3.6mm" H 7500 2450 50  0001 C CNN
+F 3 "https://www.analog.com/media/en/technical-documentation/data-sheets/AD2S1210.pdf" H 7500 2450 50  0001 C CNN
+	2    7400 2450
+	1    0    0    -1
+$EndComp
 $EndSCHEMATC
